Commit message: feat: add mission-centric excavator operator workflow
Add ROS mission actions, RViz operator panel, live and fixture planning, supervised live control, fixed dig/dump actions, right-handed frame integration, and regression coverage. Fixed-action step timeouts now fail closed instead of advancing and reporting success.

File: kinematics/waji_description/urdf/waji.urdf (robot description, URDF)
Before this commit: robot waji, 7 links, 6 joints
Joints:
- joint arm_joint: origin xyz=0.78 0 0 rpy=0 3.31 0 -> xyz=0.78 0 0 rpy=0 2.95 0
- joint boom_joint: origin xyz=0.05 0 0 rpy=0 0.43 0 -> xyz=0.05 0 0 rpy=0 0.52 0
- joint bucket_joint: origin xyz=0.35 0 0 rpy=0 3.48 0 -> xyz=0.35 0 0 rpy=0 2.74 0
